File: battery/electronics/63-00013_Battery_PCB_6.3.brd (EAGLE design)
At the start: 46 x 58.6 mm, 339 parts, among them IC1 BQ294700DSG, IC10 TPS70933DRV, IC11 BQ24780SRUY, IC14 824001, IC26 BQ769X2PFB, IC4 n.m., IC5 TMP112NAIDRL, IC6 824001, IC8 STM32G431CBU6, Q1 TSX-3225_24.0000MF10Z-C, Q2 ECS-.327-12.5-12R, T1 SISS06DN, T11 PMV30ENEA, T12 PMV30ENEA, T13 SISS06DN, T14 SISS06DN, T15 PMV30ENEA, T16 PMV30ENEA, T17 PMV30ENEA, T2 DMG1012UW-7, T3 SISS06DN, T4 PMV30ENEA, T5 PMV30ENEA, T6 PMV30ENEA, T7 DMG1012UW-7, T8 CSD17577Q3A, T9 CSD17308Q3, X1 MUSBR-M5C1-M0, X13 n.m., X14 665102131822, X2 665102131822, X21 TC2030-CTX, X6 TC2030-CTX

Commit message: updated engineering files
Parts:
- C1, C10, C102, C103, C11, C12, C13, C14, C16, C166, C167, C168, C169, C17, C170, C175, C18, C21, C29, C295, C296, C3, C36, C37, C38, C39, C4, C41, C42, C45, C46, C48, C49, C50, C53, C56, C59, C6, C60, C61, C62, C63, C64, C65, C7, C8, C9: device 03_DT_Passive_Components:C0603 -> 03_TFH_Passive_Components:C0603
- C171, C19, C20, C22, C23, C24, C25, C26, C27, C28, C30, C31, C32, C33, C34, C35: device 03_DT_Passive_Components:C1210 -> 03_TFH_Passive_Components:C1210
- C173, C177, C43, C44, C47, C52: device 03_DT_Passive_Components:C0805 -> 03_TFH_Passive_Components:C0805
- C2, C234, C235, C282, C283, C40, C5: value 100p 25V -> 100p 50V; device 03_DT_Passive_Components:C0603 -> 03_TFH_Passive_Components:C0603
- D1, D4: device 02_DT_Discrete_Semiconductors:SMA_ST -> 02_TFH_Discrete_Semiconductors:SMA_ST
- D10, D19, D5, D6, D7, D8: device 02_DT_Discrete_Semiconductors:SOD323F_SC-90_NXP -> 02_TFH_Discrete_Semiconductors:SOD323F_SC-90_NXP
- D11: device 02_DT_Discrete_Semiconductors:SOT-323_DIODES_INC -> 02_TFH_Discrete_Semiconductors:SOT-323_DIODES_INC
- D12, D13, D14, D15, D16, D17, D18, D2, D20, D3, D9: device 02_DT_Discrete_Semiconductors:150044M155260_WUERTH -> 02_TFH_Discrete_Semiconductors:150044M155260_WUERTH
- F1: device 01_DT_Fuses:0680L_BEL_FUSE -> 01_TFH_Fuses:0680L_BEL_FUSE
- F2: device 01_DT_Fuses:SFJ-XX12_DEXERIALS -> 01_TFH_Fuses:SFJ-XX12_DEXERIALS
- H1, H2: device 09_DT_Holes:2,3-PAD -> 09_TFH_Holes:2,3-PAD
- IC1: value BQ294700DSG -> BQ294703DSG; device 04_DT_Integrated_Circuits:DSG0008A_WSON_TI -> 04_TFH_Integrated_Circuits:DSG0008A_WSON_TI
- IC10: device 04_DT_Integrated_Circuits:DRV0006A_TI -> 04_TFH_Integrated_Circuits:DRV0006A_TI
- IC11: device 04_DT_Integrated_Circuits:RUY0028A_TI -> 04_TFH_Integrated_Circuits:RUY0028A_TI
- IC14, IC6: device 04_DT_Integrated_Circuits:SOT23-6L_WE -> 04_TFH_Integrated_Circuits:SOT23-6L_WE
- IC26: device 04_DT_Integrated_Circuits:S-PQFP-G48_PFB_TI -> 04_TFH_Integrated_Circuits:S-PQFP-G48_PFB_TI
- IC4: device 04_DT_Integrated_Circuits:S-PDSO-G8_DGK_VSSOP_TI -> 04_TFH_Integrated_Circuits:S-PDSO-G8_DGK_VSSOP_TI
- IC5: device 04_DT_Integrated_Circuits:DRL0006A_TI -> 04_TFH_Integrated_Circuits:DRL0006A_TI
- IC8: device 04_DT_Integrated_Circuits:UFQFPN48_ST -> 04_TFH_Integrated_Circuits:UFQFPN48_ST
- L16: device 03_DT_Passive_Components:FERRIT_1806_WUERTH -> 03_TFH_Passive_Components:FERRIT_1806_WUERTH
- L2: device 03_DT_Passive_Components:WE-PD_1260_WE -> 03_TFH_Passive_Components:WE-PD_1260_WE
- PS1, PS2, PS3, PS4, PS5, PS6: device 07_DT_Miscellaneous:PASSERMARKE -> 07_TFH_Miscellaneous:PASSERMARKE
- PTC1: device 03_DT_Passive_Components:R0402 -> 03_TFH_Passive_Components:R0402
- Q1: device 03_DT_Passive_Components:TSX-3225_SEIKO_EPSON -> 03_TFH_Passive_Components:TSX-3225_SEIKO_EPSON
- Q2: device 03_DT_Passive_Components:ECX-12R_ECS -> 03_TFH_Passive_Components:ECX-12R_ECS
- R1, R10, R100, R101, R102, R103, R104, R105, R106, R107, R108, R109, R11, R110, R111, R112, R113, R114, R115, R116, R117, R118, R12, R121, R122, R123, R124, R125, R126, R127, R128, R129, R13, R130, R131, R132, R133, R134, R135, R136, R137, R138, R139, R14, R140, R141, R142, R143, R144, R145, R146, R147, R148, R149, R15, R16, R17, R176, R177, R18, R189, R19, R190, R191, R2, R20, R21, R217, R218, R22, R227, R228, R229, R23, R232, R24, R25, R26, R27, R28, R29, R296, R3, R30, R322, R337, R34, R35, R36, R4, R41, R42, R43, R44, R45, R46, R47, R48, R49, R5, R50, R51, R52, R53, R54, R55, R56, R57, R58, R59, R6, R60, R61, R62, R63, R64, R65, R66, R67, R68, R69, R70, R71, R72, R73, R74, R75, R76, R77, R78, R79, R8, R80, R81, R82, R83, R84, R85, R86, R87, R88, R89, R9, R90, R92, R93, R94, R95, R96, R97, R98, R99: device 03_DT_Passive_Components:R0603 -> 03_TFH_Passive_Components:R0603
- R192, R37, R7: device 03_DT_Passive_Components:LVT12_R003_OHMITE -> 03_TFH_Passive_Components:LVT12_R003_OHMITE
- S1: device 05_DT_Electromechanic:430451025836_WUERTH -> 05_TFH_Electromechanic:430451025836_WUERTH
- SPACER1, SPACER2: device 05_DT_Electromechanic:702916000_WUERTH -> 05_TFH_Electromechanic:702916000_WUERTH
- T1, T13, T14, T3: device 02_DT_Discrete_Semiconductors:POWERPAK_1212-8S_VISHAY -> 02_TFH_Discrete_Semiconductors:POWERPAK_1212-8S_VISHAY
- T11, T12, T15, T16, T17, T4, T5, T6: device 02_DT_Discrete_Semiconductors:SOT-23_NXP -> 02_TFH_Discrete_Semiconductors:SOT-23_NXP
- T8: device 02_DT_Discrete_Semiconductors:Q3A_TI -> 02_TFH_Discrete_Semiconductors:Q3A_TI
- T9: device 02_DT_Discrete_Semiconductors:Q3_TI -> 02_TFH_Discrete_Semiconductors:Q3_TI
- TP1, TP10, TP11, TP17, TP18, TP2, TP23, TP24, TP25, TP26, TP27, TP28, TP29, TP3, TP30, TP31, TP32, TP33, TP34, TP35, TP36, TP37, TP38, TP39, TP4, TP40, TP41, TP42, TP43, TP5, TP6, TP7, TP8, TP9: device 07_DT_Miscellaneous:TESTVIA_ROUND_0.8MM -> 07_TFH_Miscellaneous:TESTVIA_ROUND_0.8MM
- X1: device 00_DT_Connectors:MUSBR-M5C1-XX_AMPHENOL -> 00_TFH_Connectors:MUSBR-M5C1-XX_AMPHENOL
- X10, X11, X7, X8, X9: device 00_DT_Connectors:WIREPAD_0.8X6.5MM -> 00_TFH_Connectors:WIREPAD_0.8X6.5MM
- X13: device 00_DT_Connectors:SSW-110-03-G-S-RA-LL_SAMTEC -> 00_TFH_Connectors:SSW-110-03-G-S-RA-LL_SAMTEC
- X14, X2: device 00_DT_Connectors:665102131822_WURTH -> 00_TFH_Connectors:665102131822_WURTH
- X21, X6: device 00_DT_Connectors:TC2030-IDC-FP_TAGCONNECT -> 00_TFH_Connectors:TC2030-IDC-FP_TAGCONNECT
