File: battery/electronics/63-00013_Battery_PCB_6.3.sch (EAGLE design)
At the start: 339 parts, among them IC1 BQ294700DSG, IC10 TPS70933DRV, IC11 BQ24780SRUY, IC14 824001, IC26 BQ769X2PFB, IC4 n.m., IC5 TMP112NAIDRL, IC6 824001, IC8 STM32G431CBU6, Q1 TSX-3225_24.0000MF10Z-C, Q2 ECS-.327-12.5-12R, T1 SISS06DN, T11 PMV30ENEA, T12 PMV30ENEA, T13 SISS06DN, T14 SISS06DN, T15 PMV30ENEA, T16 PMV30ENEA, T17 PMV30ENEA, T2 DMG1012UW-7, T3 SISS06DN, T4 PMV30ENEA, T5 PMV30ENEA, T6 PMV30ENEA, T7 DMG1012UW-7, T8 CSD17577Q3A, T9 CSD17308Q3, X1 MUSBR-M5C1-M0, X13 n.m., X14 665102131822, X2 665102131822, X21 TC2030-CTX, X6 TC2030-CTX

Commit message: updated engineering files
Parts:
- C1, C10, C11, C12, C13, C14, C16, C166, C167, C168, C169, C17, C170, C175, C18, C21, C29, C3, C36, C37, C38, C39, C4, C41, C42, C45, C46, C48, C49, C50, C53, C56, C59, C6, C60, C61, C62, C63, C7, C8, C9: device 03_DT_Passive_Components:C-EUC0603 -> 03_TFH_Passive_Components:C-EU-100N-C0603; VOLTAGE 50.0 V -> (none)
- C102, C103, C295, C296: device 03_DT_Passive_Components:C-EUC0603 -> 03_TFH_Passive_Components:C-EU-27P-C0603; DIELECTRIC C0G/NP0 -> (none); VOLTAGE 50.0 V -> (none)
- C171, C19, C20, C22, C23, C24, C25, C26, C27, C28, C30, C31, C32, C33, C34, C35: device 03_DT_Passive_Components:C-EUC1210 -> 03_TFH_Passive_Components:C-EU-4U7-25V-C1210; VOLTAGE 25 V -> (none)
- C173, C44: device 03_DT_Passive_Components:C-EUC0805 -> 03_TFH_Passive_Components:C-EU-1U-C0805; VOLTAGE 25.0 V -> (none)
- C177, C43, C47, C52: device 03_DT_Passive_Components:C-EUC0805 -> 03_TFH_Passive_Components:C-EU-22U-C0805; VOLTAGE 10.0 V -> (none)
- C2, C234, C235, C282, C283, C40, C5: value 100p 25V -> 100p 50V; device 03_DT_Passive_Components:C-EUC0603 -> 03_TFH_Passive_Components:C-EU-100P-C0603; VOLTAGE 25.0 V -> (none)
- C64, C65: device 03_DT_Passive_Components:C-EUC0603 -> 03_TFH_Passive_Components:C-EU-C0603
- D1, D4: device 02_DT_Discrete_Semiconductors:SMA6J20A -> 02_TFH_Discrete_Semiconductors:SMA6J20A
- D10, D19, D5, D6, D7, D8: device 02_DT_Discrete_Semiconductors:PMEG6010CEJ -> 02_TFH_Discrete_Semiconductors:PMEG6010CEJ
- D11: device 02_DT_Discrete_Semiconductors:BAS70W-05 -> 02_TFH_Discrete_Semiconductors:BAS70W-05
- D12, D13, D14, D15, D16, D17, D18, D2, D20, D3, D9: device 02_DT_Discrete_Semiconductors:150044M155260 -> 02_TFH_Discrete_Semiconductors:150044M155260
- F1: device 01_DT_Fuses:0680L9100-0 -> 01_TFH_Fuses:0680L9100-0
- F2: device 01_DT_Fuses:SFJ-1412 -> 01_TFH_Fuses:SFJ-1412
- H1, H2: device 09_DT_Holes:MOUNT-PAD-ROUND2.3 -> 09_TFH_Holes:MOUNT-PAD-ROUND2.3
- IC1: value BQ294700DSG -> BQ294703DSG; device 04_DT_Integrated_Circuits:BQ294700DSG -> 04_TFH_Integrated_Circuits:BQ294703DSG
- IC10: device 04_DT_Integrated_Circuits:TPS70933DRV -> 04_TFH_Integrated_Circuits:TPS70933DRV
- IC11: device 04_DT_Integrated_Circuits:BQ24780SRUY -> 04_TFH_Integrated_Circuits:BQ24780SRUY
- IC14, IC6: device 04_DT_Integrated_Circuits:824001 -> 04_TFH_Integrated_Circuits:824001
- IC26: device 04_DT_Integrated_Circuits:BQ769X2PFB -> 04_TFH_Integrated_Circuits:BQ769X2PFB
- IC4: device 04_DT_Integrated_Circuits:TMP1075DGK -> 04_TFH_Integrated_Circuits:TMP1075DGK
- IC5: device 04_DT_Integrated_Circuits:TMP112NAIDRL -> 04_TFH_Integrated_Circuits:TMP112NAIDRL
- IC8: device 04_DT_Integrated_Circuits:STM32G431CBU6 -> 04_TFH_Integrated_Circuits:STM32G431CBU6
- L16: device 03_DT_Passive_Components:742792410 -> 03_TFH_Passive_Components:742792410
- L2: device 03_DT_Passive_Components:744771004 -> 03_TFH_Passive_Components:744771004
- PS1, PS2, PS3, PS4, PS5, PS6: device 07_DT_Miscellaneous:PASSERMARKE -> 07_TFH_Miscellaneous:PASSERMARKE
- PTC1: device 03_DT_Passive_Components:PRF15BE103RB6RC -> 03_TFH_Passive_Components:PRF15BE103RB6RC
- Q1: device 03_DT_Passive_Components:TSX-3225_24.0000MF10Z-C -> 03_TFH_Passive_Components:TSX-3225_24.0000MF10Z-C
- Q2: device 03_DT_Passive_Components:ECS-.327-12.5-12R -> 03_TFH_Passive_Components:ECS-.327-12.5-12R
- R1, R141, R145, R146, R149, R26, R42, R56, R8, R99: device 03_DT_Passive_Components:R-EUR0603 -> 03_TFH_Passive_Components:R-EU-100K-R0603
- R10, R15, R17, R20, R21, R22, R30, R49, R9: device 03_DT_Passive_Components:R-EUR0603 -> 03_TFH_Passive_Components:R-EU-1K-R0603
- R100, R101, R103, R104, R106, R107, R109, R110, R112, R113, R115, R116, R189, R190, R191, R25, R64, R65, R70, R71, R73, R74, R76, R77: device 03_DT_Passive_Components:R-EUR0603 -> 03_TFH_Passive_Components:R-EU-150R-R0603
- R102, R105, R108, R111, R114, R228, R296, R63, R66, R72, R75, R78: device 03_DT_Passive_Components:R-EUR0603 -> 03_TFH_Passive_Components:R-EU-330R-R0603
- R11, R117, R118, R121, R122, R126, R127, R128, R129, R130, R131, R132, R133, R134, R135, R136, R137, R138, R139, R140, R142, R143, R144, R16, R176, R177, R19, R229, R23, R232, R3, R322, R337, R35, R36, R41, R44, R45, R46, R47, R51, R52, R53, R57, R58, R6, R60, R61, R62, R67, R68, R69, R92, R95: device 03_DT_Passive_Components:R-EUR0603 -> 03_TFH_Passive_Components:R-EU-10R-R0603
- R12, R123, R2, R217, R218, R227, R80, R81, R84, R85, R93, R94, R96, R97, R98: device 03_DT_Passive_Components:R-EUR0603 -> 03_TFH_Passive_Components:R-EU-10K-R0603
- R124, R125, R13, R14, R34, R43, R48, R50, R54, R79, R86, R87, R88, R89: device 03_DT_Passive_Components:R-EUR0603 -> 03_TFH_Passive_Components:R-EU-10M-R0603
- R147, R148, R18, R27, R29, R4, R5, R59, R82, R83, R90: device 03_DT_Passive_Components:R-EUR0603 -> 03_TFH_Passive_Components:R-EU-0R-R0603
- R192, R37, R7: device 03_DT_Passive_Components:LVT12R0050FER -> 03_TFH_Passive_Components:LVT12R0050FER
- R24, R28, R55: device 03_DT_Passive_Components:R-EUR0603 -> 03_TFH_Passive_Components:R-EU-510K-R0603
- S1: device 05_DT_Electromechanic:430451025836 -> 05_TFH_Electromechanic:430451025836
- SPACER1, SPACER2: device 05_DT_Electromechanic:702916000 -> 05_TFH_Electromechanic:702916000
- T1, T13, T14, T3: device 02_DT_Discrete_Semiconductors:SISS06DN -> 02_TFH_Discrete_Semiconductors:SISS06DN
- T11, T12, T15, T16, T17, T4, T5, T6: device 02_DT_Discrete_Semiconductors:PMV30ENEA -> 02_TFH_Discrete_Semiconductors:PMV30ENEA
- T8: device 02_DT_Discrete_Semiconductors:CSD17577Q3A -> 02_TFH_Discrete_Semiconductors:CSD17577Q3A
- T9: device 02_DT_Discrete_Semiconductors:CSD17308Q3 -> 02_TFH_Discrete_Semiconductors:CSD17308Q3
- TP1, TP10, TP11, TP17, TP18, TP2, TP23, TP24, TP25, TP26, TP27, TP28, TP29, TP3, TP30, TP31, TP32, TP33, TP34, TP35, TP36, TP37, TP38, TP39, TP4, TP40, TP41, TP42, TP43, TP5, TP6, TP7, TP8, TP9: device 07_DT_Miscellaneous:TESTPOINT_VIA_ROUND_0.8MM -> 07_TFH_Miscellaneous:TESTPOINT_VIA_ROUND_0.8MM
- X1: device 00_DT_Connectors:MUSBR-M5C1-M0 -> 00_TFH_Connectors:MUSBR-M5C1-M0
- X10, X11, X7, X8, X9: device 00_DT_Connectors:WIREPAD_0.8X6.5MM -> 00_TFH_Connectors:WIREPAD_0.8X6.5MM
- X13: device 00_DT_Connectors:SSW-110-03-G-S-RA-LL -> 00_TFH_Connectors:SSW-110-03-G-S-RA-LL
- X14, X2: device 00_DT_Connectors:665102131822 -> 00_TFH_Connectors:665102131822
- X21, X6: device 00_DT_Connectors:TC2030-CTX -> 00_TFH_Connectors:TC2030-CTX
Other:
- note added: "hardware versions: 6.0: R125 = 0R; R124 = n.m. 6.1 / 6.2: R125 = n.m.; R124 = 0R 6.3: R125 = 10M; R124 = 10M"
- note removed: "hardware versions: 6.0: R125 = 0R; R124 = n.m. 6.1: R125 = n.m.; R124 = 0R 6.2: R125 = 10M; R124 = 10M"
